Commit message: add walking

File: environment/urdf/ur5_suction.urdf (robot description, URDF)
Before this commit: robot ur5_robotiq_140, 10 links, 9 joints
Links:
- link gripper_surf: geometry visual box size=0.02 0.14 0.14

Commit message: teke op

File: environment/urdf/ur5_suction.urdf (robot description, URDF)
Before this commit: robot ur5_robotiq_140, 10 links, 9 joints
Links:
- link gripper_surf: geometry visual box size=0.02 0.07 0.07
